Commit message: succesfully got a reset and random action to work

File: src/bd1_description/urdf/bd1.xacro (robot description, xacro)
@@ -130,5 +130,5 @@
         <child link="head_link"/>
         <origin xyz="0 0 ${neck_len}" rpy="0 1.5 0"/>
-        <limit effort="${servo_effort}" velocity="${servo_velocity}" lower="0" upper="${pi}"/>
+        <limit effort="${servo_effort}" velocity="${servo_velocity}" lower="-${pi}" upper="${pi}"/>
         <axis xyz="0 1 0"/>
         <dynamics damping="${servo_friction}"/>
